Commit message: fix(assets): update franka-panda with gripper and gsmini robot asset
Mainly, new finger model (with cable protector and closer gap).
Asset is still for Isaac 5.1. For Isaac 6 we need to reimport the urdf and adjust the robot asset.

File: source/tacex_assets/tacex_assets/data/Robots/Franka/GelSight_Mini/franka_panda_description_w_gripper_gsmini/franka_panda_w_gripper_gsmini.urdf (robot description, URDF)
Before this commit: robot panda, 12 links, 11 joints
Links:
- link panda_hand: geometry collision mesh filename=package://franka_panda_description_w_gripper_gsmini/meshes/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; visual mesh filename=package://franka_panda_description_w_gripper_gsmini/meshes/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
- link panda_leftfinger: geometry collision mesh filename=package://franka_panda_description_w_gripper_gsmini/meshes/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; visual mesh filename=package://franka_panda_description_w_gripper_gsmini/meshes/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
- link panda_link0: geometry collision mesh filename=package://franka_panda_description_w_gripper_gsmini/meshes/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; visual mesh filename=package://franka_panda_description_w_gripper_gsmini/meshes/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
- link panda_link1: geometry collision mesh filename=package://franka_panda_description_w_gripper_gsmini/meshes/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; visual mesh filename=package://franka_panda_description_w_gripper_gsmini/meshes/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
- link panda_link2: geometry collision mesh filename=package://franka_panda_description_w_gripper_gsmini/meshes/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; visual mesh filename=package://franka_panda_description_w_gripper_gsmini/meshes/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
- link panda_link3: geometry collision mesh filename=package://franka_panda_description_w_gripper_gsmini/meshes/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; visual mesh filename=package://franka_panda_description_w_gripper_gsmini/meshes/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
- link panda_link4: geometry collision mesh filename=package://franka_panda_description_w_gripper_gsmini/meshes/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; visual mesh filename=package://franka_panda_description_w_gripper_gsmini/meshes/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
- link panda_link5: geometry collision mesh filename=package://franka_panda_description_w_gripper_gsmini/meshes/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; visual mesh filename=package://franka_panda_description_w_gripper_gsmini/meshes/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
- link panda_link6: geometry collision mesh filename=package://franka_panda_description_w_gripper_gsmini/meshes/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; visual mesh filename=package://franka_panda_description_w_gripper_gsmini/meshes/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
- link panda_link7: geometry collision mesh filename=package://franka_panda_description_w_gripper_gsmini/meshes/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; visual mesh filename=package://franka_panda_description_w_gripper_gsmini/meshes/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
- link panda_rightfinger: geometry collision mesh filename=package://franka_panda_description_w_gripper_gsmini/meshes/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; visual mesh filename=package://franka_panda_description_w_gripper_gsmini/meshes/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
